File: Test Board.kicad_pcb (KiCad board)
At the start: 2 copper layers, 43 parts, among them J1 SCREW TERMINAL, J2 SCREW TERMINAL, Q1 BT138-600, Q2 BT138-600, Q3 BT138-600, Q4 S8050, SW1 UP-MJTP1230, SW2 LT-MJTP1230, SW3 DN-MJTP1230, SW4 RT-MJTP1230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

Commit message: Finished Board Layout
Parts:
- removed Q1, Q2, Q3: BT138-600, Package_TO_SOT_THT:TO-220-3_Vertical
- removed Q4: S8050, Package_TO_SOT_THT:TO-92_Inline
- removed R10, R11, R12: 33R, Resistor_THT:R_Axial_DIN0207_L6.3mm_D2.5mm_P7.62mm_Horizontal
- removed R13, R14, R16, R17: 10k, Resistor_THT:R_Axial_DIN0207_L6.3mm_D2.5mm_P7.62mm_Horizontal
- removed R15: 4.7k, Resistor_THT:R_Axial_DIN0207_L6.3mm_D2.5mm_P7.62mm_Horizontal
- removed R2, R3: 560R, Resistor_THT:R_Axial_DIN0207_L6.3mm_D2.5mm_P7.62mm_Horizontal
- removed R4, R5, R6: 180R, Resistor_THT:R_Axial_DIN0207_L6.3mm_D2.5mm_P7.62mm_Horizontal
- removed R7, R8, R9: 100R, Resistor_THT:R_Axial_DIN0207_L6.3mm_D2.5mm_P7.62mm_Horizontal
- removed U3, U4: MOC3012M, Package_DIP:DIP-6_W7.62mm
- added C1: 680uF, Capacitor_THT:CP_Radial_D12.5mm_P5.00mm, F.Cu at (67.3, 64.8)
- added C2: 680uF, Capacitor_THT:CP_Radial_D12.5mm_P5.00mm, F.Cu at (104.8, 65.4)
- added D3: LED, LED_THT:LED_D5.0mm, F.Cu at (102.9, 76.8)
- added J3: SCREW TERMINAL, TerminalBlock_Phoenix:TerminalBlock_Phoenix_MKDS-1,5-2-5.08_1x02_P5.08mm_Horizontal, F.Cu at (45.7, 116.8)
- added K1: FINDER-32.21-x300, Relay_THT:Relay_SPST_Finder_32.21-x300, F.Cu at (76.2, 87.0)
- added K2: FINDER-32.21-x300, Relay_THT:Relay_SPST_Finder_32.21-x300, F.Cu at (76.2, 114.9)
- added K3: FINDER-32.21-x300, Relay_THT:Relay_SPST_Finder_32.21-x300, F.Cu at (76.2, 101.6)
- added R23: 220R, Resistor_THT:R_Axial_DIN0207_L6.3mm_D2.5mm_P7.62mm_Horizontal, F.Cu at (99.1, 76.8)
- D1: value B40C5000-3x00A -> D_Bridge_+AA-; footprint Diode_THT:Diode_Bridge_32.0x5.6x17.0mm_P10.0mm_P7.5mm -> Diode_THT:Diode_Bridge_Vishay_KBPM
- D2: value MBR360 -> SB5199TA
- J2: footprint TerminalBlock_Phoenix:TerminalBlock_Phoenix_MKDS-1,5-3-5.08_1x03_P5.08mm_Horizontal -> TerminalBlock_Phoenix:TerminalBlock_Phoenix_MKDS-1,5-2-5.08_1x02_P5.08mm_Horizontal
- L1: value 330uH -> 53uH; footprint Inductor_THT:L_Radial_D21.0mm_P19.00mm -> Inductor_THT:L_Toroid_Vertical_L21.6mm_W11.4mm_P7.62mm_Pulse_KM-3
- R1: value 560R -> 220R
- RV1: footprint Resistor_THT:R_Axial_DIN0207_L6.3mm_D2.5mm_P7.62mm_Horizontal -> Potentiometer_THT:Potentiometer_Bourns_3266Y_Vertical
- U1: value LM2575-5.0BT -> LM2596T-5; footprint Package_TO_SOT_THT:TO-220-5_Vertical -> Package_TO_SOT_THT:TO-220-5_P3.4x3.7mm_StaggerOdd_Lead3.8mm_Vertical
- U2: value MOC3012M -> L293D; footprint Package_DIP:DIP-6_W7.62mm -> Package_DIP:DIP-16_W7.62mm
- moved U6 102.9 mm to (190.5, 121.9), turned to 90 degrees
- moved RV1 92.3 mm to (199.4, 57.1), turned to 90 degrees
- moved DS1 85.0 mm to (123.2, 59.1)
- moved A1 82.9 mm to (104.1, 116.8), turned to 90 degrees
- moved R20 82.9 mm to (163.8, 120.7)
- moved R22 78.7 mm to (190.5, 99.1)
- moved R21 67.5 mm to (175.9, 102.2)
- moved SW4 65.5 mm to (176.5, 106.7)
- moved SW2 50.9 mm to (152.4, 106.7)
- moved R18 48.3 mm to (163.8, 97.2)
- moved R19 48.3 mm to (159.4, 102.2), turned to 180 degrees
- moved SW3 48.2 mm to (164.5, 111.8)
- moved SW1 46.9 mm to (164.5, 101.6)
- moved L1 46.3 mm to (78.1, 71.8)
- moved U2 42.3 mm to (91.4, 111.8), turned to 180 degrees
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Connections:
- A1 pad 13: Net-(A1-Pad13) -> /BKLT
- A1 pad 19: Net-(A1-Pad19) -> /E
- A1 pad 20: Net-(A1-Pad20) -> /RS
- A1 pad 21: Net-(A1-Pad21) -> /D7
- A1 pad 22: Net-(A1-Pad22) -> /D6
- A1 pad 23: SDA -> /D5
- A1 pad 24: SCL -> /D4
- D1 pad 1: GND -> +VDC
- D1 pad 2: /R -> /C
- D1 pad 3: /C -> /R
- D1 pad 4: +VDC -> GND
- DS1 pad 15: +5V -> Net-(DS1-Pad15)
- DS1 pad 16: Net-(DS1-Pad16) -> GND
- DS1 pad 5: /RW -> GND
- J2 pad 1: /W -> /G
- J2 pad 2: /G -> /Y
- R1 pad 1: Net-(R1-Pad1) -> Net-(DS1-Pad15)
- R1 pad 2: /FAN -> /BACKLIGHT
- U2 pad 1: Net-(R1-Pad1) -> +5V
- U2 pad 2: GND -> /FAN
- U2 pad 3: Net-(U2-Pad3) -> /FANRLY
- U2 pad 4: Net-(Q1-Pad3) -> GND
- U2 pad 5: Net-(U2-Pad5) -> GND
- U2 pad 6: Net-(R7-Pad2) -> /HEATRLY
Routing:
- net /DHT: track 0.00 -> 106.0 mm
- net Net-(DS1-Pad3): track 0.00 -> 74.2 mm
- net /R: track 0.00 -> 67.2 mm
- net /SW_RT: track 0.00 -> 65.1 mm
- net /COOL: track 0.00 -> 63.9 mm, vias 0 -> 1
- net /SW_UP: track 0.00 -> 61.5 mm
- net Net-(DS1-Pad15): track 0.00 -> 60.9 mm, vias 0 -> 1
- net /D7: track 0.00 -> 54.6 mm
- net /D4: track 0.00 -> 54.6 mm
- net /D6: track 0.00 -> 54.6 mm
- net /D5: track 0.00 -> 54.6 mm
- net /BKLT: track 0.00 -> 54.0 mm
- net +5V: track 0.00 -> 52.9 mm
- net /SW_DN: track 0.00 -> 51.0 mm
- net /E: track 0.00 -> 44.1 mm
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- added copper zone on B.Cu, net +5V
- added copper zone on F.Cu, net GND
Other:
- board outline added: 165.1 x 76.2 mm
- board text added: "Designed by A. Elder"
