File: Test Board.sch (KiCad schematic (older format))
At the start: 13 parts

Commit message: Finished Schematic
Parts:
- removed D?: VS-KBPC802, Diode_THT:Diode_Bridge_Vishay_KBPC6, symbol Diode_Bridge:VS-KBPC802
- removed U?: PCA8574PW, SOT403-1_NXP, symbol IOExpander:PCA8574PW
- added C3, C4, C5: 0.01uf, symbol Device:C_Small
- added C6: 220uF, symbol Device:CP
- added D1: B40C5000-3x00A, Diode_THT:Diode_Bridge_32.0x5.6x17.0mm_P10.0mm_P7.5mm, symbol Diode_Bridge:B40C5000-3x00A
- added J2: SCREW TERMINAL, symbol Connector:Screw_Terminal_01x03
- added Q1, Q2, Q3: BT138-600, Package_TO_SOT_THT:TO-220-3_Vertical, symbol Triac_Thyristor:BT138-600
- added Q4: S8050, Package_TO_SOT_THT:TO-92_Inline, symbol Transistor_BJT:S8050
- added R1, R2, R3: 560R, Resistor_THT:R_Axial_DIN0207_L6.3mm_D2.5mm_P7.62mm_Horizontal, symbol Device:R
- added R10, R11, R12: 33R, Resistor_THT:R_Axial_DIN0207_L6.3mm_D2.5mm_P7.62mm_Horizontal, symbol Device:R
- added R15: 4.7k, Resistor_THT:R_Axial_DIN0207_L6.3mm_D2.5mm_P7.62mm_Horizontal, symbol Device:R
- added R16, R22: 10k, Resistor_THT:R_Axial_DIN0207_L6.3mm_D2.5mm_P7.62mm_Horizontal, symbol Device:R
- added R18, R19, R20, R21: 47k, Resistor_THT:R_Axial_DIN0207_L6.3mm_D2.5mm_P7.62mm_Horizontal, symbol Device:R
- added R4, R5, R6: 180R, Resistor_THT:R_Axial_DIN0207_L6.3mm_D2.5mm_P7.62mm_Horizontal, symbol Device:R
- added R7, R8, R9: 100R, Resistor_THT:R_Axial_DIN0207_L6.3mm_D2.5mm_P7.62mm_Horizontal, symbol Device:R
- added RV1: 10k, Resistor_THT:R_Axial_DIN0207_L6.3mm_D2.5mm_P7.62mm_Horizontal, symbol Device:R_POT
- added SW1: UP-MJTP1230, Button_Switch_THT:SW_PUSH_6mm, symbol Switch:SW_Push
- added SW2: LT-MJTP1230, Button_Switch_THT:SW_PUSH_6mm, symbol Switch:SW_Push
- added SW3: DN-MJTP1230, Button_Switch_THT:SW_PUSH_6mm, symbol Switch:SW_Push
- added SW4: RT-MJTP1230, Button_Switch_THT:SW_PUSH_6mm, symbol Switch:SW_Push
- added U2, U3, U4: MOC3012M, symbol Relay_SolidState:MOC3012M
- added U5: PCA8574PW, SOT403-1_NXP, symbol IOExpander:PCA8574PW
- added U6: DHT11, Sensor:Aosong_DHT11_5.5x12.0_P2.54mm, symbol Sensor:DHT11
- J1: renamed from J?; value Screw_Terminal_01x02 -> SCREW TERMINAL
- R13, R14, R17: renamed from R?; footprint (none) -> Resistor_THT:R_Axial_DIN0207_L6.3mm_D2.5mm_P7.62mm_Horizontal
- gave numbers to parts that had none: 7
Connections:
- net labels added: C, COOL, DHT, FAN, G, HEAT, R, SW_DN, SW_LT, SW_RT, SW_UP, W, Y
- wire segments 32 -> 109
- no-connect marks 0 -> 22
Other:
- moved on the sheet: A1, C1, C2, D2, J1, L1, U1

Commit message: Added BOM
Parts:
- D2: footprint (none) -> Diode_THT:D_DO-201_P15.24mm_Horizontal
- J1: footprint (none) -> TerminalBlock_Phoenix:TerminalBlock_Phoenix_MKDS-1,5-2-5.08_1x02_P5.08mm_Horizontal
- J2: footprint (none) -> TerminalBlock_Phoenix:TerminalBlock_Phoenix_MKDS-1,5-3-5.08_1x03_P5.08mm_Horizontal
- L1: footprint (none) -> Inductor_THT:L_Radial_D21.0mm_P19.00mm
- U2, U3, U4: footprint (none) -> Package_DIP:DIP-6_W7.62mm
Changed lines of the file:
@@
 F 0 "D2" V 2804 1630 50  0000 L CNN
 F 1 "MBR360" V 2895 1630 50  0000 L CNN
-F 2 "" H 2850 1550 50  0001 C CNN
+F 2 "Diode_THT:D_DO-201_P15.24mm_Horizontal" H 2850 1550 50  0001 C CNN
 F 3 "~" H 2850 1550 50  0001 C CNN
 	1    2850 1550
@@
 F 0 "L1" V 3390 1400 50  0000 C CNN
 F 1 "330uH" V 3299 1400 50  0000 C CNN
-F 2 "" H 3200 1400 50  0001 C CNN
+F 2 "Inductor_THT:L_Radial_D21.0mm_P19.00mm" H 3200 1400 50  0001 C CNN
 F 3 "~" H 3200 1400 50  0001 C CNN
 	1    3200 1400
@@
 F 0 "J1" H 1568 5567 50  0000 C CNN
 F 1 "SCREW TERMINAL" H 1568 5476 50  0000 C CNN
-F 2 "" H 1650 5350 50  0001 C CNN
+F 2 "TerminalBlock_Phoenix:TerminalBlock_Phoenix_MKDS-1,5-2-5.08_1x02_P5.08mm_Horizontal" H 1650 5350 50  0001 C CNN
 F 3 "~" H 1650 5350 50  0001 C CNN
 	1    1650 5350
@@
 F 0 "J2" H 1568 5575 50  0000 C CNN
 F 1 "SCREW TERMINAL" H 1568 5666 50  0000 C CNN
-F 2 "" H 1650 5900 50  0001 C CNN
+F 2 "TerminalBlock_Phoenix:TerminalBlock_Phoenix_MKDS-1,5-3-5.08_1x03_P5.08mm_Horizontal" H 1650 5900 50  0001 C CNN
 F 3 "~" H 1650 5900 50  0001 C CNN
 	1    1650 5900
@@
 F 0 "U4" H 3800 7025 50  0000 C CNN
 F 1 "MOC3012M" H 3800 6934 50  0000 C CNN
-F 2 "" H 3600 6500 50  0001 L CIN
+F 2 "Package_DIP:DIP-6_W7.62mm" H 3600 6500 50  0001 L CIN
 F 3 "https://www.onsemi.com/pub/Collateral/MOC3023M-D.PDF" H 3800 6700 50  0001 L CNN
 	1    3800 6700
@@
 F 0 "U3" H 3800 6025 50  0000 C CNN
 F 1 "MOC3012M" H 3800 5934 50  0000 C CNN
-F 2 "" H 3600 5500 50  0001 L CIN
+F 2 "Package_DIP:DIP-6_W7.62mm" H 3600 5500 50  0001 L CIN
 F 3 "https://www.onsemi.com/pub/Collateral/MOC3023M-D.PDF" H 3800 5700 50  0001 L CNN
 	1    3800 5700
@@
 F 0 "U2" H 3800 5025 50  0000 C CNN
 F 1 "MOC3012M" H 3800 4934 50  0000 C CNN
-F 2 "" H 3600 4500 50  0001 L CIN
+F 2 "Package_DIP:DIP-6_W7.62mm" H 3600 4500 50  0001 L CIN
 F 3 "https://www.onsemi.com/pub/Collateral/MOC3023M-D.PDF" H 3800 4700 50  0001 L CNN
 	1    3800 4700

Commit message: Finished Board Layout
Parts:
- removed C3, C4, C5: 0.01uf, symbol Device:C_Small
- removed C6: 220uF, symbol Device:CP
- removed D1: B40C5000-3x00A, Diode_THT:Diode_Bridge_32.0x5.6x17.0mm_P10.0mm_P7.5mm, symbol Diode_Bridge:B40C5000-3x00A
- removed J2: SCREW TERMINAL, TerminalBlock_Phoenix:TerminalBlock_Phoenix_MKDS-1,5-3-5.08_1x03_P5.08mm_Horizontal, symbol Connector:Screw_Terminal_01x03
- removed Q1, Q2, Q3: BT138-600, Package_TO_SOT_THT:TO-220-3_Vertical, symbol Triac_Thyristor:BT138-600
- removed Q4: S8050, Package_TO_SOT_THT:TO-92_Inline, symbol Transistor_BJT:S8050
- removed R10, R11, R12: 33R, Resistor_THT:R_Axial_DIN0207_L6.3mm_D2.5mm_P7.62mm_Horizontal, symbol Device:R
- removed R13, R14, R16, R17: 10k, Resistor_THT:R_Axial_DIN0207_L6.3mm_D2.5mm_P7.62mm_Horizontal, symbol Device:R
- removed R15: 4.7k, Resistor_THT:R_Axial_DIN0207_L6.3mm_D2.5mm_P7.62mm_Horizontal, symbol Device:R
- removed R2, R3: 560R, Resistor_THT:R_Axial_DIN0207_L6.3mm_D2.5mm_P7.62mm_Horizontal, symbol Device:R
- removed R4, R5, R6: 180R, Resistor_THT:R_Axial_DIN0207_L6.3mm_D2.5mm_P7.62mm_Horizontal, symbol Device:R
- removed R7, R8, R9: 100R, Resistor_THT:R_Axial_DIN0207_L6.3mm_D2.5mm_P7.62mm_Horizontal, symbol Device:R
- removed U1: LM2575-5.0BT, Package_TO_SOT_THT:TO-220-5_Vertical, symbol Regulator_Switching:LM2575-5.0BT
- removed U2, U3, U4: MOC3012M, Package_DIP:DIP-6_W7.62mm, symbol Relay_SolidState:MOC3012M
- removed U5: PCA8574PW, SOT403-1_NXP, symbol IOExpander:PCA8574PW
- added D1: D_Bridge_+AA-, Diode_THT:Diode_Bridge_Vishay_KBPM, symbol Device:D_Bridge_+AA-
- added D3: LED, LED_THT:LED_D5.0mm, symbol Device:LED
- added J2, J3: SCREW TERMINAL, TerminalBlock_Phoenix:TerminalBlock_Phoenix_MKDS-1,5-2-5.08_1x02_P5.08mm_Horizontal, symbol Connector:Screw_Terminal_01x02
- added K1, K2, K3: FINDER-32.21-x300, Relay_THT:Relay_SPST_Finder_32.21-x300, symbol Relay:FINDER-32.21-x300
- added R23: 220R, Resistor_THT:R_Axial_DIN0207_L6.3mm_D2.5mm_P7.62mm_Horizontal, symbol Device:R
- added U1: LM2596T-5, Package_TO_SOT_THT:TO-220-5_P3.4x3.7mm_StaggerOdd_Lead3.8mm_Vertical, symbol Regulator_Switching:LM2596T-5
- added U2: L293D, Package_DIP:DIP-16_W7.62mm, symbol Driver_Motor:L293D
- C1: value 100uF -> 680uF; footprint (none) -> Capacitor_THT:CP_Radial_D12.5mm_P5.00mm
- C2: value 220uF -> 680uF; footprint (none) -> Capacitor_THT:CP_Radial_D12.5mm_P5.00mm
- D2: value MBR360 -> SB5199TA
- L1: value 330uH -> 53uH; footprint Inductor_THT:L_Radial_D21.0mm_P19.00mm -> Inductor_THT:L_Toroid_Vertical_L21.6mm_W11.4mm_P7.62mm_Pulse_KM-3
- R1: value 560R -> 220R
- RV1: footprint Resistor_THT:R_Axial_DIN0207_L6.3mm_D2.5mm_P7.62mm_Horizontal -> Potentiometer_THT:Potentiometer_Bourns_3266Y_Vertical
Connections:
- net RW is gone; now on net GND: DS1.5 (R/W)
- net SCL is gone; now on net D4: A1.24 (A5)
- net SDA is gone; now on net D5: A1.23 (A4)
- net +5V: now also D3.2 (A), U1.4 (FB), U2.1 (EN1,2), U2.16 (VCC1), U2.8 (VCC2), U2.9 (EN3,4); no longer DS1.15 (LED(+))
- net +VDC: now also D1.1 (+), U1.1 (VIN)
- net C: now also D1.2 (~~)
- net COOL: now also U2.10 (3A)
- net D6: now also A1.22 (A3)
- net D7: now also A1.21 (A2)
- net E: now also A1.19 (A0)
- net FAN: now also U2.2 (1A); no longer R1.2
- net G: now also J2.1 (Pin_1), K1.11
- net GND: now also DS1.16 (LED(-)), D1.4 (-), K1.A2, K2.A2, K3.A2, R23.2, U1.3 (GND), U1.5 (~ON~/OFF), U2.12 (GND), U2.13 (GND), U2.4 (GND), U2.5 (GND)
- net HEAT: now also U2.7 (2A)
- net R: now also D1.3 (~~), K1.14, K2.14, K3.14
- net RS: now also A1.20 (A1)
- net W: now also J3.1 (Pin_1), K2.11
- net Y: now also J2.2 (Pin_2), K3.11
- net at D2.1 (K), L1.1: now also U1.2 (OUT)
- net BKLT: now reaches A1.13 (D10)
- net BKLT: now also U2.15 (4A)
- net at R1.1: now also DS1.15 (LED(+))
- new net: D3.1 (K), R23.1
- new net BACKLIGHT: R1.2, U2.14 (4Y)
- new net COOLRLY: K3.A1, U2.11 (3Y)
- new net FANRLY: K1.A1, U2.3 (1Y)
- new net HEATRLY: K2.A1, U2.6 (2Y)
- no-connect marks 22 -> 17
Other:
- moved on the sheet: DS1, RV1

Commit message: Started working on firmware
Parts:
- A1: symbol MCU_Module:Arduino_Nano_v3.x -> Test-Board-rescue:Arduino_Nano_v3.x-MCU_Module
Changed lines of the file:
@@
 $EndComp
 $Comp
-L MCU_Module:Arduino_Nano_v3.x A1
+L Test-Board-rescue:Arduino_Nano_v3.x-MCU_Module A1
 U 1 1 6118DE62
 P 10200 1800
