File: Board/Test Board.kicad_sch (KiCad schematic)
At the start: 31 parts

Commit message: Continue V2 Design
Parts:
- added D?: D, symbol Device:D
- A1: value (none) -> Adafruit_Feather_HUZZAH_ESP8266; footprint (none) -> Module:Adafruit_Feather
- C1, C2: value (none) -> 680uF; footprint (none) -> Capacitor_THT:CP_Radial_D18.0mm_P7.50mm
- D1: value (none) -> D_Bridge_+AA-; footprint (none) -> Arduino-Thermostat:Diode Bridge 4-SMD
- D2: value (none) -> VS-50WQ04FNTR-M3; footprint (none) -> Package_TO_SOT_SMD:TO-252-3_TabPin2
- D3: value (none) -> LED; footprint (none) -> LED_THT:LED_D5.0mm
- J1, J2, J3: value (none) -> SCREW TERMINAL; footprint (none) -> TerminalBlock_Phoenix:TerminalBlock_Phoenix_MKDS-1,5-2-5.08_1x02_P5.08mm_Horizontal
- L1: value (none) -> 68uH; footprint (none) -> Inductor_THT:L_Radial_L16.1mm_W16.1mm_Px7.62mm_Py12.70mm_Pulse_LP-44
- Q1, Q2, Q3: value (none) -> Q_NMOS_GSD; footprint (none) -> Package_TO_SOT_SMD:SOT-23
- R1, R2, R3: value (none) -> 10K; footprint (none) -> Resistor_SMD:R_1206_3216Metric
- R10: value (none) -> 1.5K; footprint (none) -> Resistor_SMD:R_1206_3216Metric
- R22: value (none) -> 10k; footprint (none) -> Resistor_SMD:R_1206_3216Metric
- R23: value (none) -> 600R; footprint (none) -> Resistor_SMD:R_1206_3216Metric
- R4, R5, R6: value (none) -> 1K; footprint (none) -> Resistor_SMD:R_1206_3216Metric
- R7: value (none) -> 4.7K; footprint (none) -> Resistor_SMD:R_1206_3216Metric
- R8: value (none) -> 2.0k; footprint (none) -> Resistor_SMD:R_1206_3216Metric
- R9: value (none) -> 820R; footprint (none) -> Resistor_SMD:R_1206_3216Metric
- U1: value (none) -> LM2596S-3.3; footprint (none) -> Package_TO_SOT_SMD:TO-263-5_TabPin3
- U2: value (none) -> Adafruit-Eink-Display; footprint (none) -> Arduino-Thermostat:Adafruit-eink-display
- U3, U4, U5: value (none) -> DS1E-M-DC3V; footprint (none) -> Arduino-Thermostat:DS1E-M-DC5V
- U6: value (none) -> DHT11; footprint (none) -> Arduino-Thermostat:DHT22-Horizontal
Connections:
- net +3V3: now also D?.1 (K)
- net COOLRLY: now also D?.2 (A)

Commit message: Continue V2 Design
Parts:
- added D4, D5: D, Diode_SMD:D_SMA_Handsoldering, symbol Device:D
- D3: footprint LED_THT:LED_D5.0mm -> LED_SMD:LED_1206_3216Metric_Pad1.42x1.75mm_HandSolder
- D6: renamed from D?; footprint (none) -> Diode_SMD:D_SMA_Handsoldering
Connections:
- net +3V3: now also D4.1 (K), D5.1 (K)
- net FANRLY: now also D4.2 (A)
- net HEATRLY: now also D5.2 (A)
Other:
- moved on the sheet: C1, C2, D2, D3, R23

Commit message: Continue board layout for v2 design
Parts:
- added R11: 470R, Resistor_SMD:R_1206_3216Metric, symbol Device:R
- added SW1, SW2, SW3, SW4: SW_Push, Button_Switch_THT:SW_PUSH_6mm_H5mm, symbol Switch:SW_Push
- R8: value 2.0k -> 2.0K
- R9: value 820R -> 4.3K
Connections:
- net ADC: now also R10.2, R11.2, SW1.1; no longer U2.23 (D11)
- net DHT: now also A1.19 (IO2); no longer A1.18 (SCL/IO5)
- net FAN: now also A1.18 (SCL/IO5); no longer A1.19 (IO2)
- net GND: now also SW1.2, SW2.2, SW3.2, SW4.2
- removed net BUTTON2: R10.2, R9.1, U2.24 (D12)
- net BUTTON3: no longer names the net of U2.25 (D13)
- net BUTTON3: no longer R10.1
- new net: R9.1, SW2.1
- new net: R10.1, SW3.1
- new net: R11.1, SW4.1
- no-connect marks 30 -> 32
Other:
- moved on the sheet: R10, R22, R9, U6

Commit message: Finished board layout, updated readme
Parts:
- added F1: Fuse, Fuse:Fuseholder_Blade_Mini_Keystone_3568, symbol Device:Fuse
Connections:
- net R: now also F1.2; no longer J1.1 (Pin_1)
- new net: F1.1, J1.1 (Pin_1)
Other:
- company: (none) -> freeport7.space
- title: Arduino Thermostat -> Arduino Thermostat V2
Changed lines of the file:
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@@
   (paper "A4")
   (title_block
-    (title "Arduino Thermostat")
-    (date "2021-08-14")
+    (title "Arduino Thermostat V2")
+    (date "2022-07-11")
     (rev "A")
+    (company "freeport7.space")
     (comment 1 "Designed by A. Elder")
   )
   (junction (at 97.79 35.56) (diameter 0) (color 0 0 0 0)
   )
+  (junction (at 36.83 30.48) (diameter 0) (color 0 0 0 0)
+  )
   (junction (at 264.16 33.02) (diameter 0) (color 0 0 0 0)
   )
@@
   )
   (junction (at 153.67 165.1) (diameter 0) (color 0 0 0 0)
-  )
-  (junction (at 36.83 30.48) (diameter 0) (color 0 0 0 0)
   )
   (junction (at 72.39 45.72) (diameter 0) (color 0 0 0 0)
@@
     (stroke (width 0) (type default) (color 0 0 0 0))
   )
+  (wire (pts (xy 46.99 135.89) (xy 50.8 135.89))
+    (stroke (width 0) (type default) (color 0 0 0 0))
+  )
   (wire (pts (xy 46.99 149.86) (xy 53.34 149.86))
     (stroke (width 0) (type default) (color 0 0 0 0))
@@
     (stroke (width 0) (type default) (color 0 0 0 0))
   )
-  (wire (pts (xy 57.15 78.74) (xy 63.5 78.74))
-    (stroke (width 0) (type default) (color 0 0 0 0))
-  )
   (wire (pts (xy 204.47 44.45) (xy 193.04 44.45))
     (stroke (width 0) (type default) (color 0 0 0 0))
@@
     (stroke (width 0) (type default) (color 0 0 0 0))
   )
+  (wire (pts (xy 57.15 78.74) (xy 64.77 78.74))
+    (stroke (width 0) (type default) (color 0 0 0 0))
+  )
   (wire (pts (xy 67.31 45.72) (xy 59.69 45.72))
     (stroke (width 0) (type default) (color 0 0 0 0))
@@
     (stroke (width 0) (type default) (color 0 0 0 0))
   )
-  (wire (pts (xy 46.99 135.89) (xy 53.34 135.89))
-    (stroke (width 0) (type default) (color 0 0 0 0))
-  )
   (wire (pts (xy 96.52 114.3) (xy 87.63 114.3))
     (stroke (width 0) (type default) (color 0 0 0 0))
@@
   )
   (wire (pts (xy 46.99 147.32) (xy 53.34 147.32))
+    (stroke (width 0) (type default) (color 0 0 0 0))
+  )
+  (wire (pts (xy 58.42 135.89) (xy 63.5 135.89))
     (stroke (width 0) (type default) (color 0 0 0 0))
   )
@@
     (effects (font (size 1.27 1.27)) (justify right bottom))
   )
-  (label "R" (at 63.5 78.74 180)
+  (label "R" (at 64.77 78.74 180)
     (effects (font (size 1.27 1.27)) (justify right bottom))
   )
-  (label "R" (at 53.34 135.89 180)
+  (label "R" (at 63.5 135.89 180)
     (effects (font (size 1.27 1.27)) (justify right bottom))
   )
@@
       (effects (font (size 1.27 1.27)) (justify right))
     )
-    (property "Value" "D_Bridge_+AA-" (id 1) (at 58.2676 79.883 90)
+    (property "Value" "D_Bridge_+AA-" (id 1) (at 58.42 81.28 90)
       (effects (font (size 1.27 1.27)) (justify right))
     )
@@
     (pin "1")
   )
+  (symbol (lib_id "Device:Fuse") (at 54.61 135.89 90) (unit 1)
+    (in_bom yes) (on_board yes) (fields_autoplaced)
+    (property "Reference" "F1" (id 0) (at 54.61 131.4282 90))
+    (property "Value" "Fuse" (id 1) (at 54.61 133.9651 90))
+    (property "Footprint" "Fuse:Fuseholder_Blade_Mini_Keystone_3568" (id 2) (at 54.61 137.668 90)
+      (effects (font (size 1.27 1.27)) hide)
+    )
+    (property "Datasheet" "~" (id 3) (at 54.61 135.89 0)
+      (effects (font (size 1.27 1.27)) hide)
+    )
+    (pin "1")
+    (pin "2")
+  )
   (symbol (lib_id "power:GND") (at 212.09 143.51 0) (unit 1)
     (in_bom yes) (on_board yes)
@@
       (reference "D6") (unit 1) (value "D") (footprint "Diode_SMD:D_SMA_Handsoldering")
     )
+    (path "/990fe46e-75fc-4017-bddd-4f16ef277679"
+      (reference "F1") (unit 1) (value "Fuse") (footprint "Fuse:Fuseholder_Blade_Mini_Keystone_3568")
+    )
     (path "/00000000-0000-0000-0000-00006118966f"
